Commit message: Updated IMU position on raw3-1

File: cob_hardware_config/raw3-1/urdf/raw3-1.urdf.xacro (robot description, xacro)
@@ -53,5 +53,5 @@
    <!-- IMU brick mount on raw3-1 -->
    <joint name="imu_brick_joint" type="fixed" >
-      <origin xyz="0.402 -0.0811 0.335" rpy="0 0 0" />
+      <origin xyz="0.495 -0.06750 0.498" rpy="0 0 0" />
       <parent link="base_link" />
       <child link="imu_brick_link" />

Commit message: updated IMU position on raw3-1

File: cob_hardware_config/raw3-1/urdf/raw3-1.urdf.xacro (robot description, xacro)
@@ -53,5 +53,5 @@
    <!-- IMU brick mount on raw3-1 -->
    <joint name="imu_brick_joint" type="fixed" >
-      <origin xyz="0.495 -0.06750 0.498" rpy="0 0 0" />
+      <origin xyz="0.495 -0.06750 0.508" rpy="0 0 0" />
       <parent link="base_link" />
       <child link="imu_brick_link" />

Commit message: urdf update: softkinetic camera mount on raw3-1

File: cob_hardware_config/raw3-1/urdf/raw3-1.urdf.xacro (robot description, xacro)
@@ -72,3 +72,23 @@
     </link>
     <!-- END: IMU brick	mount -->
+    <!-- Softkinetic 'left' mount on raw3-1 -->
+    <joint name="softkinetic_left_joint" type="fixed" >
+      <origin xyz="0.495 0.06750 0.498" rpy="0 0 0" />
+      <parent link="base_link" />
+      <child link="softkinect_left_link" />
+    </joint>
+    <link name="softkinect_left_link">
+       <inertial>
+            <mass value="0.0001" />
+            <origin xyz="0 0 0" rpy="0 0 0" />
+            <inertia ixx="0.00001" ixy="0" ixz="0" iyy="0.00001" iyz="0" izz="0.00001" />
+       </inertial>
+       <visual>
+   	    <origin xyz="0 0 0" rpy="0 0 0" />
+	    <geometry>
+    	       <box size="0.03 0.10 0.05" />
+	    </geometry>
+	    <material name="IPA/LightGrey" />
+       </visual>
+    </link>
   </robot>
